File: BQ7790522PWR/BQ7790522PWR.sch (KiCad schematic (older format))
At the start: 53 parts, among them J1 BAT, J2 BAT_NEG, J3 DSG, J4 LDU, J5 LOAD_NEG, J6 TS, J7 CTRD, J8 CTRC, J9 CHGU, Q1 IAUC41N06S5N102ATMA1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

Commit message: update schematic and pcb
Parts:
- removed Q1, Q2: IAUC41N06S5N102ATMA1, BQ7790522PWR:IAUC41N06S5N102, symbol Device:Q_NMOS_GDS
- added U2, U3: SIR172ADP-T1-GE3, Package_SO:PowerPAK_SO-8_Single, symbol BQ7790522PWR:SIR172ADP-T1-GE3
- R23, R24: value 0 -> 1k
Connections:
- net B_OUT: now also U3.1 (S), U3.2 (S), U3.3 (S)
- net SW_C: now also U2.5 (D), U3.5 (D)
- net SW_IN: now also U2.1 (S), U2.2 (S), U2.3 (S)
- net at R10.2, R11.1: now also U2.4 (G)
- net at D1.1 (K), D2.1 (K), R13.2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: now also U3.4 (G)
Changed lines of the file:
@@
-$EndComp
-$Comp
-L Device:Q_NMOS_GDS Q1
-U 1 1 62A750D9
-P 3550 6850
-F 0 "Q1" V 3799 6850 50  0000 C CNN
-F 1 "IAUC41N06S5N102ATMA1" V 3900 6650 50  0000 C CNN
-F 2 "BQ7790522PWR:IAUC41N06S5N102" H 3750 6950 50  0001 C CNN
-F 3 "~" H 3550 6850 50  0001 C CNN
-	1    3550 6850
-	0    1    1    0
-$EndComp
-$Comp
-L Device:Q_NMOS_GDS Q2
-U 1 1 62A77A23
-P 4250 6850
-F 0 "Q2" V 4499 6850 50  0000 C CNN
-F 1 "IAUC41N06S5N102ATMA1" V 4600 6650 50  0000 C CNN
-F 2 "BQ7790522PWR:IAUC41N06S5N102" H 4450 6950 50  0001 C CNN
-F 3 "~" H 4250 6850 50  0001 C CNN
-	1    4250 6850
-	0    -1   1    0
 $EndComp
 $Comp
@@
 	3250 6950 3350 6950
 Wire Wire Line
-	3750 6950 4050 6950
-Wire Wire Line
 	4350 7600 4600 7600
 Wire Wire Line
@@
 $EndComp
 Wire Wire Line
-	3550 6650 3550 6600
-Wire Wire Line
-	3550 6600 3100 6600
-Wire Wire Line
 	3100 6600 3100 6550
 Wire Wire Line
@@
 	0    1    1    0
 $EndComp
-Wire Wire Line
-	4250 6650 4250 6600
-Wire Wire Line
-	4250 6600 4600 6600
 Wire Wire Line
 	4900 6600 4900 6650
@@
 P 8100 1600
 F 0 "R23" H 8041 1554 50  0000 R CNN
-F 1 "0" H 8041 1645 50  0000 R CNN
+F 1 "1k" H 8041 1645 50  0000 R CNN
 F 2 "Resistor_SMD:R_0805_2012Metric" H 8100 1600 50  0001 C CNN
 F 3 "~" H 8100 1600 50  0001 C CNN
@@
 P 8450 1600
 F 0 "R24" H 8391 1554 50  0000 R CNN
-F 1 "0" H 8391 1645 50  0000 R CNN
+F 1 "1k" H 8391 1645 50  0000 R CNN
 F 2 "Resistor_SMD:R_0805_2012Metric" H 8450 1600 50  0001 C CNN
 F 3 "~" H 8450 1600 50  0001 C CNN
@@
 Text Label 6050 6950 0    50   ~ 0
 B_OUT
-Text Label 3800 6950 0    50   ~ 0
+Text Label 2200 7250 0    50   ~ 0
 SW_C
 Text Label 2550 6950 0    50   ~ 0
@@
 Text Label 8350 2400 0    50   ~ 0
 CHGU
+$Comp
+L BQ7790522PWR:SIR172ADP-T1-GE3 U2
+U 1 1 62ADDA5E
+P 3450 6800
+F 0 "U2" H 3500 6950 50  0000 C CNN
+F 1 "SIR172ADP-T1-GE3" H 3450 6350 50  0000 C CNN
+F 2 "Package_SO:PowerPAK_SO-8_Single" H 3450 6700 50  0001 C CNN
+F 3 "" H 3450 6700 50  0001 C CNN
+	1    3450 6800
+	1    0    0    -1
+$EndComp
+$Comp
+L BQ7790522PWR:SIR172ADP-T1-GE3 U3
+U 1 1 62ADF8B0
+P 4350 6800
+F 0 "U3" H 4550 6950 50  0000 C CNN
+F 1 "SIR172ADP-T1-GE3" H 4350 6350 50  0000 C CNN
+F 2 "Package_SO:PowerPAK_SO-8_Single" H 4350 6700 50  0001 C CNN
+F 3 "" H 4350 6700 50  0001 C CNN
+	1    4350 6800
+	-1   0    0    -1
+$EndComp
+Wire Wire Line
+	3350 6900 3350 6950
+Connection ~ 3350 6950
+Wire Wire Line
+	3350 6950 3350 7000
+Wire Wire Line
+	3350 7100 3350 7000
+Connection ~ 3350 7000
+Wire Wire Line
+	3350 6800 3350 6600
+Wire Wire Line
+	3350 6600 3100 6600
+Wire Wire Line
+	4450 6800 4450 6600
+Wire Wire Line
+	4450 6600 4600 6600
+Wire Wire Line
+	4450 6900 4450 6950
+Connection ~ 4450 6950
+Wire Wire Line
+	4450 6950 4450 7000
+Connection ~ 4450 7000
+Wire Wire Line
+	4450 7000 4450 7100
+Text Label 3900 6950 1    50   ~ 0
+SW_C
+Wire Wire Line
+	3800 6950 4000 6950
 $EndSCHEMATC
